File: KiCad/Power_Amplifier/Power Amplifier Rod Elltior Project 3A.kicad_pcb (KiCad board)
At the start: 2 copper layers, 136 x 124.5 mm, 64 parts, among them J1 AUDIO IN, J10 +35V, J11 -35V, J2 GND, J3 +35V, J4 -35V, J5 SPEAKER OUT, J6 V+, J7 COM, J8 V-, J9 GND, Q1 BC546, Q2 BC546, Q3 BC546, Q4 BD140 MJE15035, Q5 BD139 MJE15034, Q6 BD140 MJE15035, Q7 2SA1943-O, Q8 2SC5200-O, Q9 BC546

Commit message: Add files via upload
Parts:
- C12, C13: footprint Capacitor_THT:CP_Radial_D10.0mm_P2.50mm -> Capacitor_THT:C_Disc_D5.0mm_W2.5mm_P2.50mm
