File: KiCad/Power_Amplifier/Power Amplifier Rod Elltior Project 3A.kicad_pcb (KiCad board)
At the start: 2 copper layers, 136 x 124.5 mm, 64 parts, among them J1 AUDIO IN, J10 +35V, J11 -35V, J2 GND, J3 +35V, J4 -35V, J5 SPEAKER OUT, J6 V+, J7 COM, J8 V-, J9 GND, Q1 BC546, Q2 BC546, Q3 BC546, Q4 BD140 MJE15035, Q5 BD139 MJE15034, Q6 BD140 MJE15035, Q7 2SA1943-O, Q8 2SC5200-O, Q9 BC546

Commit message: Add files via upload
Parts:
- moved J5 81.4 mm to (206.8, 66.8)
Routing:
- net Net-(J5-Pin_1): track 115.3 -> 114.6 mm
Changed lines of the file:
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@@
 	(footprint "Connector_Wire:SolderWire-6sqmm_1x01_D3.5mm_OD7mm"
 		(layer "F.Cu")
-		(at 127.5 85.5)
+		(at 206.75 66.75)
 		(descr "Soldered wire connection, for a single 6 mm² wire, reinforced insulation, conductor diameter 3.5mm, outer diameter 7mm, size source Multi-Contact FLEXI-xV 2.5 (https://www.staubli.com/content/dam/ecs/catalogs-brochures/TM/CAB-Main-11014119-en.pdf#page=11), bend radius 3 times outer diameter")
 		(tags "connector wire 6sqmm")
@@
 	)
 	(segment
-		(start 194 68.5)
-		(end 193.34 68.5)
+		(start 196.66 68.5)
+		(end 205 68.5)
 		(width 2.5)
 		(layer "F.Cu")
@@
 	)
 	(segment
-		(start 193.34 68.5)
-		(end 184.34 59.5)
+		(start 205 68.5)
+		(end 206.75 66.75)
 		(width 2.5)
 		(layer "F.Cu")
@@
 	)
 	(segment
-		(start 187.92 74.92)
-		(end 187.92 74.58)
+		(start 194 68.5)
+		(end 193.34 68.5)
 		(width 2.5)
 		(layer "F.Cu")
@@
 	)
 	(segment
-		(start 155.5 83)
-		(end 164 83)
+		(start 193.34 68.5)
+		(end 184.34 59.5)
 		(width 2.5)
 		(layer "F.Cu")
@@
 	)
 	(segment
-		(start 138.184785 87.5)
-		(end 129.5 87.5)
+		(start 187.92 74.92)
+		(end 187.92 74.58)
 		(width 2.5)
 		(layer "F.Cu")
@@
 	)
 	(segment
-		(start 129.5 87.5)
-		(end 127.5 85.5)
+		(start 155.5 83)
+		(end 164 83)
 		(width 2.5)
 		(layer "F.Cu")

Commit message: Add files via upload
Parts:
- R13, R14: footprint Resistor_THT:R_Axial_DIN0516_L15.5mm_D5.0mm_P20.32mm_Horizontal -> Resistor_THT:R_Axial_Power_L25.0mm_W9.0mm_P30.48mm
- moved J5 3.40 mm to (209.5, 68.8)
- moved R14 1.60 mm to (205.2, 80.0)
- moved C8 1.25 mm to (176.2, 73.2)
Routing:
- net Net-(Q5-E): track 38.4 -> 28.5 mm
- net Net-(J5-Pin_1): track 114.6 -> 110.6 mm, vias 4 -> 3
- net Net-(C8-Pad1): track 6.04 -> 4.91 mm
- net Net-(Q6-E): track 47.7 -> 47.0 mm
