File: KiCad/Power_Amplifier/power_supply.kicad_sch (KiCad schematic)
At the start: 13 parts, among them J10 +35V, J11 -35V, J6 V+, J7 COM, J8 V-, J9 GND

Commit message: Add files via upload
Parts:
- C12, C13: footprint Capacitor_THT:CP_Radial_D10.0mm_P2.50mm -> Capacitor_THT:C_Disc_D5.0mm_W2.5mm_P2.50mm
Changed lines of the file:
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@@
 			)
 		)
-		(property "Footprint" "Capacitor_THT:CP_Radial_D10.0mm_P2.50mm"
+		(property "Footprint" "Capacitor_THT:C_Disc_D5.0mm_W2.5mm_P2.50mm"
 			(at 103.8352 95.25 0)
 			(hide yes)
@@
 			)
 		)
-		(property "Footprint" "Capacitor_THT:CP_Radial_D10.0mm_P2.50mm"
+		(property "Footprint" "Capacitor_THT:C_Disc_D5.0mm_W2.5mm_P2.50mm"
 			(at 116.5352 95.25 0)
 			(hide yes)
