File: KiCad/Power_Amplifier/power_amplifier.kicad_sch (KiCad schematic)
At the start: 46 parts, among them J1 AUDIO IN, J2 GND, J3 +35V, J4 -35V, J5 SPEAKER OUT, Q1 BC546, Q2 BC546, Q3 BC546, Q4 BD140 MJE15035, Q5 BD139 MJE15034, Q6 BD140 MJE15035, Q7 2SA1943-O, Q8 2SC5200-O, Q9 BC546

Commit message: Add files via upload
Parts:
- R13, R14: footprint Resistor_THT:R_Axial_DIN0516_L15.5mm_D5.0mm_P20.32mm_Horizontal -> Resistor_THT:R_Axial_Power_L25.0mm_W9.0mm_P30.48mm
Changed lines of the file:
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@@
 			)
 		)
-		(property "Footprint" "Resistor_THT:R_Axial_DIN0516_L15.5mm_D5.0mm_P20.32mm_Horizontal"
+		(property "Footprint" "Resistor_THT:R_Axial_Power_L25.0mm_W9.0mm_P30.48mm"
 			(at 151.384 120.396 90)
 			(hide yes)
@@
 			)
 		)
-		(property "Footprint" "Resistor_THT:R_Axial_DIN0516_L15.5mm_D5.0mm_P20.32mm_Horizontal"
+		(property "Footprint" "Resistor_THT:R_Axial_Power_L25.0mm_W9.0mm_P30.48mm"
 			(at 151.384 98.806 90)
 			(hide yes)
