File: KiCad/Power Amplifier/Power Amplifier Rod Elliot Project 3A.kicad_pcb (KiCad board)
At the start: 2 copper layers, 136 x 124.5 mm, 64 parts, among them J1 AUDIO IN, J10 +35V, J11 -35V, J2 GND, J3 +35V, J4 -35V, J5 SPEAKER OUT, J6 V+, J7 COM, J8 V-, J9 GND, Q1 BC546, Q2 BC546, Q3 BC546, Q4 BD140 MJE15035, Q5 BD139 MJE15034, Q6 BD140 MJE15035, Q7 2SA1943-O, Q8 2SC5200-O, Q9 BC546

Commit message: Add files via upload
Parts:
- Q7: value 2SA1943-O -> MJL21193G
- Q8: value 2SC5200-O -> MJL21194G
- R1, R10, R11, R12, R16, R2, R3, R4, R5, R6, R7, R8, R9: footprint Resistor_THT:R_Axial_DIN0204_L3.6mm_D1.6mm_P7.62mm_Horizontal -> Resistor_THT:R_Axial_DIN0207_L6.3mm_D2.5mm_P10.16mm_Horizontal
- moved R12 3.04 mm to (167.0, 54.7)
- moved R9 2.85 mm to (158.0, 64.3)
- moved R4 2.76 mm to (128.0, 79.8)
- moved R8 2.57 mm to (113.4, 74.8)
- moved R2 2.46 mm to (113.4, 71.5)
- moved R5 2.23 mm to (147.0, 70.2)
- moved R6 1.02 mm to (133.0, 55.2)
- moved C6 0.25 mm to (159.2, 77.8)
Routing:
- net Net-(J5-Pin_1): track 110.6 -> 90.5 mm, vias 3 -> 1
- net Net-(C5-Pad2): track 32.0 -> 40.3 mm
- net Net-(Q2-C): track 224.5 -> 228.1 mm
- net SIGNAL_GND: track 23.9 -> 20.7 mm
- net Net-(Q4-C): track 103.1 -> 105.6 mm
- net Net-(Q5-C): track 75.2 -> 72.8 mm
- net Net-(Q1-B): track 11.3 -> 13.5 mm
- net Net-(Q6-C): track 103.6 -> 101.6 mm
- net Net-(Q1-C): track 37.0 -> 38.3 mm
- net Net-(Q3-E): track 12.9 -> 14.1 mm
- net Net-(Q2-B): track 26.0 -> 26.9 mm
- net Net-(C3-Pad2): track 12.2 -> 13.1 mm
- net Net-(D1-A): track 14.7 -> 15.5 mm
- net Net-(D1-K): track 281.1 -> 281.8 mm
- net Net-(C2-Pad1): track 28.4 -> 28.9 mm
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